File: hardware/currentsense.kicad_sch (KiCad schematic)
At the start: 10 parts, among them U701 MAX49925, U703 MAX49925

Commit message: first mod
Parts:
- C701, C702, C703, C704, R702, R704, U701, U703: now not fitted; now left out of the parts list
Changed lines of the file:
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@@
 		(unit 1)
 		(exclude_from_sim no)
-		(in_bom yes)
-		(on_board yes)
-		(dnp no)
+		(in_bom no)
+		(on_board no)
+		(dnp yes)
 		(property "Reference" "C702"
 			(at 162.56 50.8063 0)
@@
 		(unit 1)
 		(exclude_from_sim no)
-		(in_bom yes)
-		(on_board yes)
-		(dnp no)
+		(in_bom no)
+		(on_board no)
+		(dnp yes)
 		(fields_autoplaced yes)
 		(property "Reference" "R702"
@@
 		(unit 1)
 		(exclude_from_sim no)
-		(in_bom yes)
-		(on_board yes)
-		(dnp no)
+		(in_bom no)
+		(on_board no)
+		(dnp yes)
 		(fields_autoplaced yes)
 		(property "Reference" "U701"
@@
 		(unit 1)
 		(exclude_from_sim no)
-		(in_bom yes)
-		(on_board yes)
-		(dnp no)
+		(in_bom no)
+		(on_board no)
+		(dnp yes)
 		(fields_autoplaced yes)
 		(property "Reference" "R704"
@@
 		(unit 1)
 		(exclude_from_sim no)
-		(in_bom yes)
-		(on_board yes)
-		(dnp no)
+		(in_bom no)
+		(on_board no)
+		(dnp yes)
 		(property "Reference" "C704"
 			(at 162.56 102.8763 0)
@@
 		(unit 1)
 		(exclude_from_sim no)
-		(in_bom yes)
-		(on_board yes)
-		(dnp no)
+		(in_bom no)
+		(on_board no)
+		(dnp yes)
 		(property "Reference" "C703"
 			(at 148.59 102.8763 0)
@@
 		(unit 1)
 		(exclude_from_sim no)
-		(in_bom yes)
-		(on_board yes)
-		(dnp no)
+		(in_bom no)
+		(on_board no)
+		(dnp yes)
 		(fields_autoplaced yes)
 		(property "Reference" "U703"
@@
 		(unit 1)
 		(exclude_from_sim no)
-		(in_bom yes)
-		(on_board yes)
-		(dnp no)
+		(in_bom no)
+		(on_board no)
+		(dnp yes)
 		(property "Reference" "C701"
 			(at 148.59 50.8063 0)

Commit message: more mods
Parts:
- removed C701, C702, C703, C704: 100n, Capacitor_SMD:C_0402_1005Metric, symbol Device:C_Small
- removed R702, R704: 0R, Resistor_SMD:R_0402_1005Metric, symbol Device:R_Small_US
- removed U701, U703: MAX49925, Package_DFN_QFN:DFN-10-1EP_3x3mm_P0.5mm_EP1.75x2.7mm, symbol matei:MAX49925
- added R1, R6: 1k5, Resistor_SMD:R_0402_1005Metric, symbol Device:R_Small_US
- added R2, R4: 22k, Resistor_SMD:R_0402_1005Metric, symbol Device:R_Small_US
- added R3, R5: 2k2, Resistor_SMD:R_0402_1005Metric, symbol Device:R_Small_US
Connections:
- net U_OUT is gone; now on net GND: R701.2
- net V_OUT is gone; now on net GND: R703.2
- net +3V3: now also R2.2, R4.2
- net GND: now also R3.1, R5.1
- net U_IN renamed SENSEA
- net SENSEA: now also R1.2
- net V_IN renamed SENSEB
- net SENSEB: now also R6.2
- new net: R4.1, R5.2
- new net: R2.1, R3.2
- new net V_SENSEA: R1.1
- new net V_SENSEB: R6.1
Other:
- note removed: "Gain 50V/V 2.9 / 50 => 58mV full range 2 * 0.020 => 40mV 0.04 * 2 = 80mW"
- note removed: "V = IR 2.9V ADC VRefBuff /20 => 0.145V input R = 0.145V/2A => 72m sense resistor P = 0.145 * 2 => 300mW rating"
- moved on the sheet: R701, R703
