File: hardware/halfbridges.kicad_sch (KiCad schematic)
At the start: 7 parts, among them U601 L6226QTR

Commit message: first mod
Parts:
- D602, D603: LCSC ID C2128 -> C81598
Changed lines of the file:
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@@
 			)
 		)
-		(property "LCSC ID" "C2128"
+		(property "LCSC ID" "C81598"
 			(at 139.7 58.42 0)
 			(effects
@@
 			)
 		)
-		(property "LCSC ID" "C2128"
+		(property "LCSC ID" "C81598"
 			(at 139.7 68.58 0)
 			(effects
@@
 			(at 107.95 99.06 0)
 			(effects
+				(font
+					(size 1.27 1.27)
+				)
+				(hide yes)
+			)
+		)
+		(property "LCSC" ""
+			(at 107.95 99.06 0)
+			(effects

Commit message: more mods
Connections:
- net GND: no longer U601.12 (SENSEB), U601.29 (SENSEA)
- new net SENSEA: U601.29 (SENSEA)
- new net SENSEB: U601.12 (SENSEB)
Changed lines of the file:
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@@
-	)
-	(junction
-		(at 158.75 114.3)
-		(diameter 0)
-		(color 0 0 0 0)
 	)
 	(junction
@@
 	)
 	(junction
-		(at 158.75 105.41)
-		(diameter 0)
-		(color 0 0 0 0)
-	)
-	(junction
 		(at 158.75 68.58)
 		(diameter 0)
@@
 	(wire
 		(pts
-			(xy 156.21 105.41) (xy 158.75 105.41)
-		)
-		(stroke
-			(width 0)
-			(type default)
-		)
-	)
-	(wire
-		(pts
 			(xy 118.11 105.41) (xy 115.57 105.41)
 		)
@@
 	(wire
 		(pts
-			(xy 158.75 105.41) (xy 158.75 114.3)
-		)
-		(stroke
-			(width 0)
-			(type default)
-		)
-	)
-	(wire
-		(pts
 			(xy 92.71 96.52) (xy 92.71 99.06)
 		)
@@
 	(wire
 		(pts
-			(xy 156.21 102.87) (xy 158.75 102.87)
+			(xy 156.21 105.41) (xy 167.64 105.41)
 		)
 		(stroke
@@
 	(wire
 		(pts
-			(xy 158.75 102.87) (xy 158.75 105.41)
+			(xy 156.21 102.87) (xy 167.64 102.87)
 		)
 		(stroke
@@
 		)
 	)
+	(hierarchical_label "SENSEB"
+		(shape output)
+		(at 167.64 105.41 0)
+		(fields_autoplaced yes)
+		(effects
+			(font
+				(size 1.27 1.27)
+			)
+			(justify left)
+		)
+	)
 	(hierarchical_label "OUT2B"
 		(shape output)
 		(at 167.64 95.25 0)
+		(fields_autoplaced yes)
+		(effects
+			(font
+				(size 1.27 1.27)
+			)
+			(justify left)
+		)
+	)
+	(hierarchical_label "SENSEA"
+		(shape output)
+		(at 167.64 102.87 0)
 		(fields_autoplaced yes)
 		(effects
@@
 		)
 		(property "LCSC ID" "C95357"
+			(at 137.16 91.44 0)
+			(effects
+				(font
+					(size 1.27 1.27)
+				)
+				(hide yes)
+			)
+		)
+		(property "Sim.Type" ""
 			(at 137.16 91.44 0)
 			(effects
@@
 			)
 		)
+		(property "Sim.Type" ""
+			(at 97.79 99.06 0)
+			(effects
+				(font
+					(size 1.27 1.27)
+				)
+				(hide yes)
+			)
+		)
 		(pin "1"
 		)
@@
 		)
 		(property "LCSC ID" "C81598"
+			(at 139.7 58.42 0)
+			(effects
+				(font
+					(size 1.27 1.27)
+				)
+				(hide yes)
+			)
+		)
+		(property "Sim.Type" ""
 			(at 139.7 58.42 0)
 			(effects
@@
 			)
 		)
+		(property "Sim.Type" ""
+			(at 149.86 68.58 0)
+			(effects
+				(font
+					(size 1.27 1.27)
+				)
+				(hide yes)
+			)
+		)
 		(pin "1"
 		)
@@
 		)
 		(property "LCSC ID" "C15195"
+			(at 129.54 63.5 0)
+			(effects
+				(font
+					(size 1.27 1.27)
+				)
+				(hide yes)
+			)
+		)
+		(property "Sim.Type" ""
 			(at 129.54 63.5 0)
 			(effects
@@
 			)
 		)
+		(property "Sim.Type" ""
+			(at 139.7 68.58 0)
+			(effects
+				(font
+					(size 1.27 1.27)
+				)
+				(hide yes)
+			)
+		)
 		(pin "1"
 		)
@@
 			(at 107.95 99.06 0)
 			(effects
+				(font
+					(size 1.27 1.27)
+				)
+				(hide yes)
+			)
+		)
+		(property "Sim.Type" ""
+			(at 107.95 99.06 0)
+			(effects
