File: hardware/lemon-pepper.kicad_pcb (KiCad board)
At the start: 4 copper layers, 35 x 35 mm, 87 parts, among them J101 INPUT, J201 USB_C_Receptacle_USB2.0, J301 TagConnect, J302 USER CONN., M101 MOT, Q501 MMBT5551, SW301 USER, U201 SRV05-4, U301 STM32G431, U302 SN65HVD230, U401 MT6835, U501 MAX15062AATA+T, U601 L6226QTR, U701 MAX49925, U703 MAX49925, Y301 12MHz

Commit message: first mod
Parts:
- removed C501, C503: 10u, Capacitor_SMD:C_0805_2012Metric
- removed C502: 1u, Capacitor_SMD:C_0402_1005Metric
- removed C701, C702, C703, C704: 100n, Capacitor_SMD:C_0402_1005Metric
- removed D501, D502: BZT52C30S, Diode_SMD:D_SOD-323
- removed JP101: TERM, Resistor_SMD:R_0402_1005Metric
- removed L501: 33u, easyeda2kicad:IND-SMD_L4.0-W4.0
- removed Q501: MMBT5551, Package_TO_SOT_SMD:SOT-23
- removed R103: 120R, Resistor_SMD:R_0402_1005Metric
- removed R501, R702, R704: 0R, Resistor_SMD:R_0402_1005Metric
- removed R504: 5R, Resistor_SMD:R_0603_1608Metric
- removed R505: 15k, Resistor_SMD:R_0402_1005Metric
- removed R506: 0R, Resistor_SMD:R_0603_1608Metric
- removed U302: SN65HVD230, Package_SO:SOIC-8_3.9x4.9mm_P1.27mm
- removed U501: MAX15062AATA+T, easyeda2kicad:TDFN-8_L2.0-W2.0-P0.50-BL
- removed U701, U703: MAX49925, Package_DFN_QFN:DFN-10-1EP_3x3mm_P0.5mm_EP1.75x2.7mm
- added C1: 1u, Capacitor_SMD:C_0402_1005Metric, F.Cu at (148.8, 110.5)
- added C2: 1u, Capacitor_SMD:C_0402_1005Metric, F.Cu at (148.8, 112.5)
- added C3: 10u, Capacitor_SMD:C_0805_2012Metric, F.Cu at (144.4, 115.7)
- added U2: XC6206PxxxMR, Package_TO_SOT_SMD:SOT-23-3, F.Cu at (144.7, 111.9)
- SW301: value USER -> BOOT0
Connections:
- net /usb/USB_5V renamed USB_5V
- R305 pad 1: /mcu/USER_BTN -> /mcu/BOOT0
- SW301 pad 1: /mcu/USER_BTN -> /mcu/BOOT0
- U301 pad 4: /mcu/USER_BTN -> unconnected-(U301-PC15-Pad4)
- U301 pad 46: /mcu/CAN_TX -> /mcu/BOOT0
- U301 pad 47: /mcu/CAN_RX -> unconnected-(U301-PB9-Pad47)
Routing:
- net /mcu/USER_BTN: track 35.6 -> 0.00 mm, vias 2 -> 0
- net /current sense/V_SENSE: track 29.9 -> 0.00 mm, vias 2 -> 0
- net /mcu/CAN_RX: track 26.9 -> 0.00 mm, vias 2 -> 0
- net /current sense/GAIN_0: track 19.5 -> 0.00 mm, vias 3 -> 0
- net /current sense/GAIN_1: track 18.9 -> 0.00 mm, vias 2 -> 0
- net /mcu/CAN_TX: track 18.0 -> 0.00 mm, vias 2 -> 0
- net /current sense/U_SENSE: track 16.8 -> 0.00 mm, vias 2 -> 0
- net +3V3: track 74.8 -> 61.7 mm, vias 17 -> 15
- net Vmot: track 24.6 -> 15.5 mm
- net Net-(C503-Pad1): track 8.09 -> 0.00 mm
- net GND: track 132.9 -> 129.1 mm
- net Net-(U501-LX): track 3.79 -> 0.00 mm
- net Net-(Q501-B): track 3.66 -> 0.00 mm
- net /current sense/U_OUT: track 6.79 -> 3.20 mm
- net /current sense/V_OUT: track 6.43 -> 2.92 mm
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
Commit message: more mods
Parts:
- added R1: 1k5, Resistor_SMD:R_0402_1005Metric, F.Cu at (146.1, 82.5)
- added R2: 22k, Resistor_SMD:R_0402_1005Metric, F.Cu at (172.7, 82.2)
- added R3: 2k2, Resistor_SMD:R_0402_1005Metric, F.Cu at (172.7, 84.2)
- added R4: 22k, Resistor_SMD:R_0402_1005Metric, F.Cu at (172.7, 86.2)
- added R5: 2k2, Resistor_SMD:R_0402_1005Metric, F.Cu at (172.7, 88.2)
- added R6: 1k5, Resistor_SMD:R_0402_1005Metric, F.Cu at (172.7, 90.2)
- H101: footprint mechanical:NEMA14 -> mechanical:NEMA17
- moved C3 34.2 mm to (171.8, 95.2)
- moved U2 16.7 mm to (146.1, 95.2)
Connections:
- net /mcu/CANH renamed /CANH
- net /mcu/CANL renamed /CANL
- M101 pad 1: /current sense/U_OUT -> /half bridges/OUT1B
- M101 pad 2: /current sense/W_IN -> /half bridges/OUT2A
- M101 pad 3: /half bridges/OUT1B -> /half bridges/OUT1A
- M101 pad 4: /current sense/V_OUT -> /half bridges/OUT2B
- R701 pad 1: /current sense/U_IN -> /current sense/SENSEA
- R701 pad 2: /current sense/U_OUT -> GND
- R703 pad 1: /current sense/V_IN -> /current sense/SENSEB
- R703 pad 2: /current sense/V_OUT -> GND
- U301 pad 11: /current sense/U_SENSE -> /current sense/V_SENSEB
- U301 pad 2: /current sense/GAIN_0 -> unconnected-(U301-PC13-Pad2)
- U301 pad 26: /current sense/V_SENSE -> /current sense/V_SENSEA
- U301 pad 3: /current sense/GAIN_1 -> unconnected-(U301-PC14-Pad3)
- U601 pad 12: GND -> /current sense/SENSEB
- U601 pad 19: /current sense/W_IN -> /half bridges/OUT2B
- U601 pad 23: /current sense/U_IN -> /half bridges/OUT2A
- U601 pad 29: GND -> /current sense/SENSEA
- U601 pad 31: /current sense/V_IN -> /half bridges/OUT1A
Routing:
- net /current sense/W_IN: track 15.6 -> 0.00 mm, vias 2 -> 0
- net /current sense/U_IN: track 15.2 -> 0.00 mm
- net /current sense/V_IN: track 11.7 -> 0.00 mm
- net /half bridges/OUT1B: track 10.8 -> 2.86 mm
- net USB_5V: track 6.01 -> 11.9 mm, vias 5 -> 6
- net GND: track 129.1 -> 123.8 mm
- net /current sense/U_OUT: track 3.20 -> 0.00 mm
- net /current sense/V_OUT: track 2.92 -> 0.00 mm
- net /CANH: track 15.4 -> 13.1 mm
- net +3V3: track 61.7 -> 63.8 mm
Other:
- board size 35 x 35 mm -> 42 x 42 mm
