File: hardware/lemon-pepper.kicad_sch (KiCad schematic)
At the start: 21 parts, among them J101 INPUT, M101 MOT

Commit message: first mod
Parts:
- R103: now not fitted; now left out of the parts list
Changed lines of the file:
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@@
 		(unit 1)
 		(exclude_from_sim no)
-		(in_bom yes)
-		(on_board yes)
-		(dnp no)
+		(in_bom no)
+		(on_board no)
+		(dnp yes)
 		(property "Reference" "R103"
 			(at 55.88 109.22 0)
@@
 		(exclude_from_sim no)
 		(in_bom no)
-		(on_board yes)
+		(on_board no)
 		(dnp yes)
 		(property "Reference" "JP101"

Commit message: more mods
Parts:
- H101: footprint mechanical:NEMA14 -> mechanical:NEMA17
Connections:
- net current sense/U_OUT is gone; now on net half bridges/OUT1B: M101.1
- net half bridges/OUT1B: no longer M101.3
- net current sense/V_OUT renamed half bridges/OUT2B
- net current sense/W_OUT renamed half bridges/OUT2A
- new net half bridges/OUT1A: M101.3
Other:
- sheet current sense ports: added SENSEA, SENSEB, V_SENSEA, V_SENSEB; removed GAIN_0, GAIN_1, U_IN, U_OUT, U_SENSE, V_IN, V_OUT, V_SENSE, W_IN, W_OUT
- sheet half bridges ports: added SENSEA, SENSEB; removed none
- sheet mcu ports: added none; removed GAIN_0, GAIN_1
- moved on the sheet: FID101, FID102, FID103, H101, M101
