File: hardware/mcu.kicad_sch (KiCad schematic)
At the start: 22 parts, among them J301 TagConnect, J302 USER CONN., SW301 USER, U301 STM32G431, U302 SN65HVD230, Y301 12MHz

Commit message: first mod
Parts:
- J301: now not fitted
- SW301: value USER -> BOOT0
- U302: now not fitted; now left out of the parts list
Connections:
- net CAN_RX: no longer U301.47 (PB9)
- net CAN_TX: no longer U301.46 (PB8)
- net USER_BTN renamed BOOT0
- net BOOT0: now also U301.46 (PB8); no longer U301.4 (PC15)
- no-connect marks 7 -> 8
Changed lines of the file:
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@@
 	)
 	(no_connect
+		(at 76.2 104.14)
+	)
+	(no_connect
 		(at 76.2 111.76)
 	)
@@
 	(wire
 		(pts
-			(xy 66.04 132.08) (xy 76.2 132.08)
-		)
-		(stroke
-			(width 0)
-			(type default)
-		)
-	)
-	(wire
-		(pts
 			(xy 143.51 58.42) (xy 143.51 59.69)
 		)
@@
 	(wire
 		(pts
-			(xy 66.04 104.14) (xy 76.2 104.14)
+			(xy 66.04 129.54) (xy 76.2 129.54)
 		)
 		(stroke
@@
 	(wire
 		(pts
-			(xy 66.04 129.54) (xy 76.2 129.54)
-		)
-		(stroke
-			(width 0)
-			(type default)
-		)
-	)
-	(wire
-		(pts
 			(xy 207.01 101.6) (xy 207.01 104.14)
 		)
@@
 		)
 	)
-	(label "CAN_RX"
-		(at 66.04 132.08 0)
-		(fields_autoplaced yes)
-		(effects
-			(font
-				(size 1.27 1.27)
-			)
-			(justify left bottom)
-		)
-	)
 	(label "TIM4_CH2"
 		(at 236.22 132.08 0)
@@
 		)
 	)
-	(label "CAN_TX"
+	(label "BOOT0"
 		(at 66.04 129.54 0)
 		(fields_autoplaced yes)
@@
 		)
 	)
-	(label "USER_BTN"
-		(at 66.04 104.14 0)
-		(fields_autoplaced yes)
-		(effects
-			(font
-				(size 1.27 1.27)
-			)
-			(justify left bottom)
-		)
-	)
 	(label "USBD_N"
 		(at 111.76 99.06 0)
@@
 		)
 	)
-	(label "USER_BTN"
+	(label "BOOT0"
 		(at 177.8 137.16 0)
 		(fields_autoplaced yes)
@@
 		(fields_autoplaced yes)
 		(property "Reference" "SW301"
-			(at 212.09 133.35 90)
+			(at 212.09 133.3499 90)
 			(effects
 				(font
@@
 			)
 		)
-		(property "Value" "USER"
-			(at 212.09 135.89 90)
+		(property "Value" "BOOT0"
+			(at 212.09 135.8899 90)
 			(effects
 				(font
@@
 		(in_bom no)
 		(on_board yes)
-		(dnp no)
+		(dnp yes)
 		(fields_autoplaced yes)
 		(property "Reference" "J301"
@@
 		(unit 1)
 		(exclude_from_sim no)
-		(in_bom yes)
-		(on_board yes)
-		(dnp no)
+		(in_bom no)
+		(on_board no)
+		(dnp yes)
 		(fields_autoplaced yes)
 		(property "Reference" "U302"

Commit message: more mods
Parts:
- removed J301: TagConnect, Connector:Tag-Connect_TC2030-IDC-NL_2x03_P1.27mm_Vertical, symbol Connector:Conn_ARM_SWD_TagConnect_TC2030-NL
- removed U302: SN65HVD230, Package_SO:SOIC-8_3.9x4.9mm_P1.27mm, symbol Interface_CAN_LIN:SN65HVD230
Connections:
- net GAIN_0: no longer names the net of U301.2 (PC13)
- net GAIN_1: no longer names the net of U301.3 (PC14)
