File: hardware/psu.kicad_sch (KiCad schematic)
At the start: 14 parts, among them Q501 MMBT5551, U501 MAX15062AATA+T

Commit message: first mod
Parts:
- added C1, C2: 1u, Capacitor_SMD:C_0402_1005Metric, symbol Device:C_Small
- added C3: 10u, Capacitor_SMD:C_0805_2012Metric, symbol Device:C_Small
- added U2: XC6206PxxxMR, Package_TO_SOT_SMD:SOT-23-3, symbol Regulator_Linear:XC6206PxxxMR
- C501, C502, C503, D501, D502, L501, Q501, R501, R504, R505, R506, U501: now not fitted; now left out of the parts list
Connections:
- net +3V3: now also C2.1, C3.1, U2.2 (VO)
- net GND: now also C1.2, C2.2, C3.2, U2.1 (GND)
- new net USB_5V: C1.1, U2.3 (VI)

Commit message: more mods
Parts:
- removed C501, C503: 10u, Capacitor_SMD:C_0805_2012Metric, symbol Device:C_Small
- removed C502: 1u, Capacitor_SMD:C_0402_1005Metric, symbol Device:C_Small
- removed D501, D502: BZT52C30S, Diode_SMD:D_SOD-323, symbol Device:D_Zener
- removed L501: 33u, easyeda2kicad:IND-SMD_L4.0-W4.0, symbol Device:L_Small
- removed Q501: MMBT5551, Package_TO_SOT_SMD:SOT-23, symbol Transistor_BJT:MMBT5551L
- removed R501: 0R, Resistor_SMD:R_0402_1005Metric, symbol Device:R_Small_US
- removed R502: 51k, Resistor_SMD:R_0402_1005Metric, symbol Device:R_Small_US
- removed R503: 22k, Resistor_SMD:R_0402_1005Metric, symbol Device:R_Small_US
- removed R504: 5R, Resistor_SMD:R_0603_1608Metric, symbol Device:R_Small_US
- removed R505: 15k, Resistor_SMD:R_0402_1005Metric, symbol Device:R_Small_US
- removed R506: 0R, Resistor_SMD:R_0603_1608Metric, symbol Device:R_Small_US
- removed U501: MAX15062AATA+T, easyeda2kicad:TDFN-8_L2.0-W2.0-P0.50-BL, symbol easyeda2kicad:MAX15062CATA+T
Connections:
- no-connect marks 1 -> 0
Other:
- note removed: "60V breakdown"
- note removed: "For MAX15062AATA+T (C2846801): R501: 0R R502, R503: DNP For MAX15062CATA+T (C1121853): R501: 200k R502, R503: 51k, 22k Ra = Rb(Vout/0.9 - 1) 3.36V (closest to 3v3 with basic parts)"
- note removed: "V = IR R = 60V/0.005 = 12K"
- moved on the sheet: C1, C2, C3, U2
